Commit message: fix the mesh to have tip at origin

File: urdf/phasma.urdf.xacro (robot description, xacro)
@@ -5,5 +5,5 @@
   <link name="base" />
   <xacro:alphasense parent="base">
-    <origin xyz="-65.210e-3 -0.109e-3 177.0e-3" rpy="0 0 0" />
+    <origin xyz="-65.253e-3 0.0 177.0e-3" rpy="0 0 0" />
   </xacro:alphasense>
   <link name="body">
@@ -20,5 +20,5 @@
   </joint>
   <xacro:hesai_device parent="base">
-    <origin xyz="-59.957e-3 0.015e-3 93.0e-3" rpy="0 0 0"/>
+    <origin xyz="-60.0e-3 0.0 93.0e-3" rpy="0 0 0"/>
   </xacro:hesai_device>
 </robot>

Commit message: load calibration from yaml

File: urdf/phasma.urdf.xacro (robot description, xacro)
@@ -3,7 +3,8 @@
   <xacro:include filename="$(find alphasense_description)/urdf/alphasense.urdf.xacro" />
   <xacro:include filename="$(find hesai_description)/urdf/hesai.urdf.xacro" />
-  <link name="base" />
-  <xacro:alphasense parent="base">
-    <origin xyz="-65.253e-3 0.0 177.0e-3" rpy="0 0 0" />
+  <link name="tip" />
+  <xacro:property name="alphasense_calibration" value="$(find phasma_description)/urdf/calibrations/20220322_calibration.yaml" />
+  <xacro:alphasense parent="tip" calib_file="${alphasense_calibration}">
+    <origin xyz="-65.253e-3 0.0 179.0e-3" rpy="0 0 0" />
   </xacro:alphasense>
   <link name="body">
@@ -14,11 +15,19 @@
     </visual>
   </link>
-  <joint name="body_to_base_mount" type="fixed">
-    <origin xyz="0 0 0" rpy="0 0 0" />
-    <parent link="base" />
+  <joint name="tip_to_body" type="fixed">
+    <origin xyz="0.0 0.0 0.0" rpy="0.0 0.0 0.0" />
+    <parent link="tip" />
     <child link="body" />
   </joint>
-  <xacro:hesai_device parent="base">
-    <origin xyz="-60.0e-3 0.0 93.0e-3" rpy="0 0 0"/>
+  <!-- This is the frame in which the ground truth is generated -->
+  <link name="base"/>
+  <!-- The base frame is coincident with the alphasense IMU but with the usual robot convention -->
+  <joint name="alphasense_imu_to_base" type="fixed">
+    <origin xyz="0.0 0.0 0.0" rpy="${-pi} 0.0 0.0" />
+    <parent link="alphasense_imu"/>
+    <child link="base"/>
+  </joint>
+  <xacro:hesai_device parent="tip">
+    <origin xyz="-60.0e-3 0.0 95.0e-3" rpy="0 0 0"/>
   </xacro:hesai_device>
 </robot>

Commit message: ros2 changes

File: urdf/phasma.urdf.xacro (robot description, xacro)
@@ -13,8 +13,8 @@
 -->
 <robot name="phasma" xmlns:xacro="http://www.ros.org/wiki/xacro">
-  <xacro:include filename="$(find alphasense_description)/urdf/alphasense.urdf.xacro" />
-  <xacro:include filename="$(find hesai_description)/urdf/hesai.urdf.xacro" />
+  <xacro:include filename="$(find-pkg-share alphasense_description)/urdf/alphasense.urdf.xacro" />
+  <xacro:include filename="$(find-pkg-share hesai_description)/urdf/hesai.urdf.xacro" />
   <link name="tip" />
-  <xacro:property name="alphasense_calibration" value="$(find phasma_description)/urdf/calibrations/20220322_calibration.yaml" />
+  <xacro:property name="alphasense_calibration" value="$(find-pkg-share phasma_description)/urdf/calibrations/20220322_calibration.yaml" />
   <xacro:alphasense parent="tip" calib_file="${alphasense_calibration}">
     <origin xyz="-65.253e-3 0.0 179.0e-3" rpy="0 0 0" />
@@ -23,5 +23,5 @@
     <visual>
       <geometry>
-        <mesh filename="package://phasma_description/urdf/meshes/phasma_body.dae" />
+        <mesh filename="$(find-pkg-share phasma_description)/urdf/meshes/phasma_body.dae" />
       </geometry>
     </visual>
